File: hardware/odsci.kicad_pcb (KiCad board)
At the start: 4 copper layers, 50 x 70 mm, 35 parts, among them J1 USB_C_Receptacle, J2 Conn_01x03_Pin, J3 Conn_01x04_Pin, J4 Screw_Terminal_01x03, SW1 SW_Push, U1 TPS7A4701xRGW, U2 STM32F042K6Tx, U3 USBLC6-2SC6

Commit message: hardware: fix position of LEDs on the pcb to match enclosure
Parts:
- moved R6 3.02 mm to (167.0, 107.9)
- moved R8 3.02 mm to (167.0, 87.9)
- moved R7 3.02 mm to (167.0, 96.8)
- moved D1 2.68 mm to (171.8, 107.3)
- moved D2 2.68 mm to (171.8, 97.3)
- moved D3 2.68 mm to (171.8, 87.3)
Routing:
- net ACTIVITY_LED: track 11.4 -> 15.9 mm
- net Net-(D3-A): track 3.00 -> 2.21 mm
- net Net-(D1-A): track 3.00 -> 2.21 mm
- net Net-(D2-A): track 3.00 -> 2.22 mm
